File: hardware/hc11main/hc11main.kicad_pcb (KiCad board)
At the start: 2 copper layers, 100 x 71 mm, 31 parts, among them P1 CONN_2X20, U10 74LS10, U11 27256, U12 74LS245, U13 74LS245, U2 68HC11A0_PLCC, U3 74LS573, U4 74LS138, U5 74LS245, U6 74LS00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

Commit message: main board: continue routing
Parts:
- added C18: 1uF, hc11:0805_m2012, F.Cu at (63.8, 43.2)
- added JP1: Jumper3, hc11:SMDPADS_3, F.Cu at (18.5, 64.8)
- added JP2: Jumper3, hc11:SMDPADS_3, F.Cu at (18.5, 66.8)
- added JP5: Jumper, hc11:SMDPADS_2, F.Cu at (68.0, 31.0)
- added JP6: Jumper, hc11:SMDPADS_2, F.Cu at (69.8, 31.0)
- added R10: 10k, hc11:0805_m2012, F.Cu at (46.5, 51.0)
- added R11: 10k, hc11:0805_m2012, F.Cu at (50.0, 49.8)
- added R12: 10k, hc11:0805_m2012, F.Cu at (46.5, 48.2)
- added R13: 10k, hc11:0805_m2012, F.Cu at (50.0, 47.0)
- added R15: 100k, hc11:0805_m2012, B.Cu at (70.0, 28.0)
- added R16: 100k, hc11:0805_m2012, B.Cu at (67.8, 28.0)
- added R17: 100k, hc11:0805_m2012, F.Cu at (105.8, 30.5)
- added R18: 100k, hc11:0805_m2012, F.Cu at (103.5, 31.2)
- added R19: 100k, hc11:0805_m2012, F.Cu at (86.3, 34.0)
- added R4: 4k7, hc11:0805_m2012, B.Cu at (21.8, 36.2)
- added R5: 4k7, hc11:0805_m2012, B.Cu at (19.8, 36.3)
- added R6: 10k, hc11:0805_m2012, F.Cu at (46.5, 56.5)
- added R7: 10k, hc11:0805_m2012, F.Cu at (50.0, 55.2)
- added R8: 10k, hc11:0805_m2012, F.Cu at (46.5, 53.8)
- added R9: 10k, hc11:0805_m2012, F.Cu at (50.0, 52.5)
- added U1: 74LS138, hc11:SOIC-16_3.9x9.9mm_P1.27mm, F.Cu at (39.4, 24.4)
- added U15: 62256, hc11:DIP-28_W15.24mm_Socket, F.Cu at (75.1, 38.1)
- R3: moved to F.Cu
- moved C11 23.4 mm to (53.8, 18.8)
- moved C9 18.9 mm to (86.5, 31.8)
- moved R3 10.6 mm to (22.0, 65.5)
- moved C12 10.2 mm to (100.7, 49.2), turned to 180 degrees
- moved C10 10.0 mm to (100.8, 43.2), turned to 180 degrees
- moved C7 9.91 mm to (100.8, 63.8), turned to 180 degrees
- moved C6 6.22 mm to (102.8, 80.2), turned to 180 degrees
- moved C15 5.76 mm to (24.2, 69.3)
- moved C16 5.76 mm to (33.2, 69.3)
- moved C17 5.76 mm to (41.8, 69.3)
- moved U10 5.76 mm to (39.2, 76.2)
- moved U6 5.76 mm to (21.8, 76.2)
- moved U7 5.76 mm to (30.8, 76.2)
- moved U11 5.39 mm to (56.0, 38.0)
- moved R1 4.83 mm to (41.0, 36.2), turned to 180 degrees
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Connections:
- net Net-(C1-Pad1) renamed /EXTAL
- net Net-(C2-Pad1) renamed /XTAL
- net Net-(R3-Pad2) renamed /MODA
- net Net-(U2-Pad4) renamed /AS
- net Net-(U2-Pad43) renamed /AN0
- net Net-(U2-Pad44) renamed /AN2
- net Net-(U2-Pad45) renamed /AN4
- net Net-(U2-Pad46) renamed /AN6
- net Net-(U2-Pad47) renamed /AN1
- net Net-(U2-Pad48) renamed /AN3
- net Net-(U2-Pad49) renamed /AN5
- net Net-(U2-Pad50) renamed /AN7
- U13 pad 19: Net-(U13-Pad19) -> /~CSEXT
- U2 pad 2: Net-(JP1-Pad2) -> /MODB
- U8 pad 20: /A15 -> /~CSRAM
Routing:
- net GND: track 55.0 -> 215.5 mm, vias 2 -> 9
- net VCC: track 31.4 -> 179.5 mm, vias 1 -> 4
- net /A13: track 0.00 -> 139.5 mm, vias 0 -> 5
- net /A10: track 10.8 -> 121.9 mm
- net /A14: track 0.00 -> 106.8 mm, vias 0 -> 3
- net /A11: track 10.6 -> 117.3 mm, vias 1 -> 3
- net /A8: track 0.00 -> 100.7 mm, vias 0 -> 1
- net /D6: track 0.00 -> 100.2 mm, vias 0 -> 3
- net /A9: track 0.00 -> 92.7 mm, vias 0 -> 2
- net /D1: track 0.00 -> 92.6 mm, vias 0 -> 2
- net /D2: track 0.00 -> 92.3 mm, vias 0 -> 2
- net /D0: track 0.00 -> 89.7 mm, vias 0 -> 2
- net /D3: track 0.00 -> 89.7 mm, vias 0 -> 1
- net /D4: track 0.00 -> 88.2 mm, vias 0 -> 2
- net /A12: track 11.0 -> 97.8 mm, vias 1 -> 3
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- added copper zone on B.Cu, net GND
- added copper zone on F.Cu, net GND
Other:
- net class Default: clearance 0.175 -> 0.25
- rule trace_clearance: 0.175 -> 0.25

Commit message: almost completed routing
Parts:
- added C19: 100n, hc11:0805_m2012, B.Cu at (79.0, 22.5)
- added C20: 100n, hc11:0805_m2012, B.Cu at (79.0, 25.8)
- added C21: 100n, hc11:0805_m2012, B.Cu at (48.5, 81.0)
- added C22: 100u, hc11:CP_Radial_D6.3mm_P2.50mm, F.Cu at (100.0, 26.8)
- added C23: 100u, hc11:CP_Radial_D6.3mm_P2.50mm, F.Cu at (51.0, 34.8)
- added C24: 47u, hc11:CP_Radial_D5.0mm_P2.00mm, F.Cu at (92.5, 76.5)
- added C25: 47u, hc11:CP_Radial_D5.0mm_P2.00mm, F.Cu at (26.8, 66.2)
- added C3: 100n, hc11:0805_m2012, F.Cu at (26.8, 28.2)
- added J1: SPI, hc11:PinHeader_2x07_P2.54mm_Vertical, F.Cu at (47.2, 22.5)
- added J2: CONN_I2C, hc11:PinHeader_1x03_P2.54mm_Vertical, F.Cu at (25.5, 21.0)
- added J3: CONN_PWR, hc11:PinHeader_1x02_P2.54mm_Vertical, F.Cu at (103.0, 21.0)
- added J4: CONN_LED, hc11:PinHeader_1x02_P2.54mm_Vertical, F.Cu at (64.2, 21.0)
- added J5: CONN_UART, hc11:PinHeader_1x03_P2.54mm_Vertical, F.Cu at (59.2, 21.0)
- added JP3: A13, hc11:SMDPADS_2, F.Cu at (93.2, 42.0)
- added JP7: A14/VPP, hc11:SMDPADS_2, F.Cu at (74.5, 33.2)
- added R14: 1k, hc11:0805_m2012, B.Cu at (59.5, 36.3)
- added R20: RSMALL, hc11:0805_m2012, B.Cu at (64.2, 24.7)
- added R21: 10k, hc11:0805_m2012, B.Cu at (40.2, 60.5)
- added T1: BS170/2N7000 (SOT23), hc11:SOT23GDS, F.Cu at (24.0, 28.8)
- added T2: BS170/2N7000 (SOT23), hc11:SOT23GDS, F.Cu at (18.5, 28.8)
- added U16: 7805, Package_TO_SOT_THT:TO-220-3_Horizontal_TabDown, F.Cu at (76.2, 21.5)
- added U17: OSC_DIL14, hc11:DIP-OSCILLATOR, F.Cu at (52.2, 80.8)
- added X1: 8 MHz, hc11:Crystal_HC49-U_Vertical, F.Cu at (39.8, 67.0)
- C11, C16, C17, C9, R19: moved to B.Cu
- moved C11 22.8 mm to (71.2, 33.4), turned to 90 degrees
- moved R19 8.87 mm to (78.0, 37.2), turned to 180 degrees
- moved U1 8.86 mm to (33.2, 30.8), turned to 90 degrees
- moved C2 7.45 mm to (34.8, 63.8), turned to 90 degrees
- moved C9 4.20 mm to (90.2, 33.5), turned to 270 degrees
- moved R15 3.86 mm to (66.2, 29.0)
- moved R16 3.62 mm to (64.2, 29.0)
- moved C18 3.51 mm to (67.2, 43.0)
- moved JP5 2.37 mm to (67.2, 33.2), turned to 270 degrees
- moved JP6 2.30 mm to (69.2, 33.2), turned to 270 degrees
- moved C10 2.25 mm to (100.8, 41.0)
- moved C1 1.98 mm to (40.0, 63.8), turned to 90 degrees
- moved R4 1.46 mm to (22.5, 35.0)
- moved R5 1.30 mm to (19.8, 35.0)
- moved C4 1.00 mm to (30.0, 48.0)
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Connections:
- P1 pad 9: /b~CSRAM -> /b~CSXRAM
- U1 pad 8: Net-(U1-Pad8) -> GND
- U15 pad 26: /A13 -> Net-(JP3-Pad1)
- U2 pad 27: /drSDA -> /SPIA2
- U2 pad 28: /drSCL -> /SPIA1
- U2 pad 30: /SPIA1 -> /drSDA
- U2 pad 31: /SPIA2 -> /drSCL
Routing:
- net GND: track 215.5 -> 632.6 mm, vias 9 -> 46
- net VCC: track 179.5 -> 437.5 mm, vias 4 -> 26
- net /E: track 24.2 -> 187.7 mm
- net /R~W: track 40.1 -> 173.2 mm, vias 2 -> 3
- net /~CSXRAM: track 27.7 -> 116.3 mm, vias 0 -> 2
- net /~CPURST: track 0.00 -> 88.1 mm, vias 0 -> 4
- net /AS: track 29.3 -> 113.8 mm, vias 0 -> 3
- net /A11: track 117.3 -> 194.9 mm, vias 3 -> 8
- net /~IRQ: track 0.00 -> 75.4 mm, vias 0 -> 2
- net /~XIRQ: track 0.00 -> 73.0 mm, vias 0 -> 2
- net /A10: track 121.9 -> 194.1 mm, vias 1 -> 7
- net /A12: track 97.8 -> 168.9 mm, vias 3 -> 7
- net /~CSROM: track 0.00 -> 51.3 mm, vias 0 -> 2
- net /~WR: track 57.0 -> 102.8 mm, vias 1 -> 5
- net /~RD: track 56.6 -> 98.7 mm, vias 0 -> 2
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- added copper zone on B.Cu, net (none)
- added copper zone on F.Cu, net (none)
- removed copper zone on B.Cu, net GND
- removed copper zone on F.Cu, net GND
Other:
- rule trace_min: 0.2 -> 0.25
- board text added: "<-RX"
- board text added: "GND"
- board text added: "I2C"
- board text added: "LED"
- board text added: "PWRLED"
- board text added: "SCL"
- board text added: "SDA"
- board text added: "SPI"
- board text added: "TX->"
- board text added: "UART"
